File: swd-multi-adapter.kicad_pcb (KiCad board)
At the start: 2 copper layers, 25.4 x 63.5 mm, 6 parts, among them J1 SWD, J2 STDC14, J3 SWD, J4 JTAG, SW1 Reset

Commit message: Added license info
Parts:
- added REF**: Symbol_CC-ShareAlike_CopperTop_Small, Symbol:Symbol_CC-ShareAlike_CopperTop_Small, B.Cu at (132.8, 120.4)
- added REF**: Symbol_CC-Attribution_CopperTop_Small, Symbol:Symbol_CC-Attribution_CopperTop_Small, B.Cu at (139.7, 120.4)
- added REF**: Symbol_CreativeCommons_CopperTop_Type2_Small, Symbol:Symbol_CreativeCommons_CopperTop_Type2_Small, B.Cu at (146.7, 120.4)
- moved REF** 0.25 mm to (143.8, 73.7)

Commit message: Added licensing info to the project files
Parts:
- removed the REF** at (132.8, 120.4)
- removed the REF** at (139.7, 120.4)
- removed the REF** at (146.7, 120.4)
Other:
- board text added: "CC BY-SA 4.0"
